File: Leiterplatte/Melodieklingel_FA86.kicad_pcb (KiCad board)
At the start: 2 copper layers, 100 x 100 mm, 45 parts

Commit message: Leiterplatte v2, mit Korrekturen
Connections:
- D100 pad 5: Net-(R101-Pad1) -> Net-(D100-Pad5)
- R101 pad 1: Net-(R101-Pad1) -> Net-(D100-Pad6)
- TP102 pad 1: Net-(D100-Pad6) -> Net-(D100-Pad5)
Routing:
- net Net-(D100-Pad6): track 6.48 -> 14.1 mm
- net Net-(D100-Pad5): track 0.00 -> 7.43 mm
- net Net-(R101-Pad1): track 4.78 -> 0.00 mm
Other:
- board text added: "29.11.2022 boert v2"
- board text removed: "11/2022 boert"
Changed lines of the file:
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@@
   (title_block
     (title "Melodieklingel")
-    (date "15.11.22")
-    (rev "1")
+    (date "29.11.22")
+    (rev "2")
     (company "FA 4/86")
     (comment 1 "boert")
@@
   (net 65 "Net-(D100-Pad6)")
   (net 66 "Net-(R100-Pad2)")
-  (net 67 "Net-(R101-Pad1)")
+  (net 67 "Net-(D100-Pad5)")
   (footprint "Resistor_THT:R_Axial_DIN0207_L6.3mm_D2.5mm_P15.24mm_Horizontal" (layer "F.Cu")
     (at 132.08 128.27 180)
@@
     (fp_line (start 1.75 1.75) (end 1.75 -1.75) (layer "F.CrtYd") (width 0.05))
     (pad "1" thru_hole rect (at 0 0) (size 2.5 2.5) (drill 1.2) (layers *.Cu *.Mask)
-      (net 65 "Net-(D100-Pad6)") (pinfunction "1") (pintype "passive"))
+      (net 67 "Net-(D100-Pad5)") (pinfunction "1") (pintype "passive"))
   )
   (footprint "RFT_sonstiges:CP_Axial_L21.0mm_D8.0mm_P28.00mm_Horizontal" (layer "F.Cu")
@@
     (fp_circle (center 0 0) (end 1.25 0) (layer "F.Fab") (width 0.1) (fill none))
     (pad "1" thru_hole circle (at 0 0 180) (size 1.6 1.6) (drill 0.8) (layers *.Cu *.Mask)
-      (net 67 "Net-(R101-Pad1)") (pintype "passive"))
+      (net 65 "Net-(D100-Pad6)") (pintype "passive"))
     (pad "2" thru_hole oval (at 5.08 0 180) (size 1.6 1.6) (drill 0.8) (layers *.Cu *.Mask)
       (net 1 "GND") (pintype "passive"))
@@
       (effects (font (size 1 1) (thickness 0.15)))
     )
-    (fp_text value "470nF" (at 7.5 4.75 90) (layer "F.Fab")
+    (fp_text value "470pF" (at 7.5 4.75 90) (layer "F.Fab")
       (effects (font (size 1 1) (thickness 0.15)))
     )
@@
       (net 1 "GND") (pintype "passive"))
     (pad "5" thru_hole oval (at 7.62 2.54 180) (size 2.4 1.6) (drill 0.8) (layers *.Cu *.Mask)
-      (net 67 "Net-(R101-Pad1)") (pintype "passive"))
+      (net 67 "Net-(D100-Pad5)") (pintype "passive"))
     (pad "6" thru_hole oval (at 7.62 0 180) (size 2.4 1.6) (drill 0.8) (layers *.Cu *.Mask)
       (net 65 "Net-(D100-Pad6)") (pintype "passive"))
@@
     (effects (font (size 1.5 1.5) (thickness 0.15)))
   )
-  (gr_text "11/2022\nboert" (at 116.84 59.944) (layer "F.SilkS")
+  (gr_text "29.11.2022\nboert\nv2" (at 116.84 59.944) (layer "F.SilkS")
     (effects (font (size 1.5 1.5) (thickness 0.15)))
   )
@@
   (segment (start 162.56 149.86) (end 161.29 148.59) (width 0.4) (layer "B.Cu") (net 63))
   (segment (start 165.1 149.86) (end 162.56 149.86) (width 0.4) (layer "B.Cu") (net 63))
-  (segment (start 156.21 147.305) (end 149.86 148.59) (width 0.4) (layer "B.Cu") (net 65))
+  (segment (start 154.94 140.462) (end 157.226 140.462) (width 0.4) (layer "B.Cu") (net 65))
+  (segment (start 158.242 146.304) (end 156.21 147.305) (width 0.4) (layer "B.Cu") (net 65))
+  (segment (start 152.175 142.24) (end 154.94 140.462) (width 0.4) (layer "B.Cu") (net 65))
+  (segment (start 157.226 140.462) (end 158.242 141.478) (width 0.4) (layer "B.Cu") (net 65))
+  (segment (start 158.242 141.478) (end 158.242 146.304) (width 0.4) (layer "B.Cu") (net 65))
   (segment (start 185.42 144.78) (end 190.5 144.78) (width 0.4) (layer "B.Cu") (net 66))
   (segment (start 181.61 148.59) (end 185.42 144.78) (width 0.4) (layer "B.Cu") (net 66))
+  (segment (start 156.21 144.765) (end 149.86 148.59) (width 0.4) (layer "B.Cu") (net 67))
   (segment (start 156.21 144.765) (end 156.195 144.78) (width 0.4) (layer "B.Cu") (net 67))
-  (segment (start 156.195 144.78) (end 152.175 142.24) (width 0.4) (layer "B.Cu") (net 67))
   (zone (net 1) (net_name "GND") (layer "F.Cu") (hatch edge 0.508)
     (connect_pads (clearance 0.508))

Commit message: fix: VT2, Footprint
Parts:
- Q: renamed from VT2; footprint Package_TO_SOT_THT:TO-39-3 -> Package_TO_SOT_THT:TO-5-3
- moved Q 5.17 mm to (186.7, 108.0), turned to 90 degrees
Connections:
- Q pad 1: Net-(R11-Pad1) -> GND
- Q pad 3: GND -> Net-(R11-Pad1)
Routing:
- net Net-(R10-Pad2): track 11.0 -> 5.84 mm
Other:
- board text added: "28.12.2022 boert v3"
- board text removed: "29.11.2022 boert v2"
Changed lines of the file:
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@@
   (title_block
     (title "Melodieklingel")
-    (date "29.11.22")
-    (rev "2")
+    (date "28.12.22")
+    (rev "3")
     (company "FA 4/86")
     (comment 1 "boert")
@@
     )
   )
-  (footprint "Package_TO_SOT_THT:TO-39-3" (layer "F.Cu")
-    (at 186.69 102.87 -90)
-    (descr "TO-39-3")
-    (tags "TO-39-3")
-    (property "Datasheet" "")
-    (property "Reference" "VT2")
+  (footprint "Package_TO_SOT_THT:TO-5-3" (layer "F.Cu")
+    (at 186.69 108.04 90)
+    (descr "TO-5-3")
+    (tags "TO-5-3")
+    (property "Datasheet" "https://www.tu-chemnitz.de/etit/zentral/ddr/sf126.gif")
+    (property "Reference" "Q")
     (property "Sheetfile" "Melodieklingel_FA86.kicad_sch")
     (property "Sheetname" "")
     (property "Value" "SF126")
     (attr through_hole)
-    (fp_text reference "VT2" (at 2.63 -6.81 180) (layer "F.SilkS")
-      (effects (font (size 1 1) (thickness 0.15)))
-    )
-    (fp_text value "SF126" (at 3.175 -7.62 180) (layer "F.Fab")
-      (effects (font (size 1 1) (thickness 0.15)))
-    )
-    (fp_text user "${REFERENCE}" (at 2.54 -0.635 180) (layer "F.Fab")
-      (effects (font (size 1 1) (thickness 0.15)))
-    )
+    (fp_text reference "VT2" (at 4.54 6.81 180) (layer "F.SilkS")
+      (effects (font (size 1 1) (thickness 0.15)))
+    )
+    (fp_text value "SF126" (at 2.54 7.81 180) (layer "F.Fab")
+      (effects (font (size 1 1) (thickness 0.15)))
+    )
+    (fp_text user "${REFERENCE}" (at 4.04 6.81 180) (layer "F.Fab")
+      (effects (font (size 1 1) (thickness 0.15)))
+    )
+    (fp_line (start -2.125856 -3.888039) (end -1.234902 -2.997084) (layer "F.SilkS") (width 0.12))
     (fp_line (start -1.348039 -4.665856) (end -2.125856 -3.888039) (layer "F.SilkS") (width 0.12))
     (fp_line (start -0.457084 -3.774902) (end -1.348039 -4.665856) (layer "F.SilkS") (width 0.12))
-    (fp_line (start -2.125856 -3.888039) (end -1.234902 -2.997084) (layer "F.SilkS") (width 0.12))
     (fp_arc (start -0.457084 -3.774902) (mid 5.948125 3.408384) (end -1.234674 -2.997371) (layer "F.SilkS") (width 0.12))
     (fp_line (start 7.49 -4.95) (end -2.41 -4.95) (layer "F.CrtYd") (width 0.05))
+    (fp_line (start -2.41 -4.95) (end -2.41 4.95) (layer "F.CrtYd") (width 0.05))
     (fp_line (start -2.41 4.95) (end 7.49 4.95) (layer "F.CrtYd") (width 0.05))
-    (fp_line (start -2.41 -4.95) (end -2.41 4.95) (layer "F.CrtYd") (width 0.05))
     (fp_line (start 7.49 4.95) (end 7.49 -4.95) (layer "F.CrtYd") (width 0.05))
     (fp_line (start -1.27151 -4.419621) (end -1.879621 -3.81151) (layer "F.Fab") (width 0.1))
@@
     (fp_arc (start -0.465408 -3.61352) (mid 5.863443 3.323361) (end -1.073594 -3.005319) (layer "F.Fab") (width 0.1))
     (fp_circle (center 2.54 0) (end 6.79 0) (layer "F.Fab") (width 0.1) (fill none))
-    (pad "1" thru_hole oval (at 0 0 270) (size 1.6 1.2) (drill 0.7) (layers *.Cu *.Mask)
+    (pad "1" thru_hole oval (at 0 0 90) (size 1.6 1.2) (drill 0.7) (layers *.Cu *.Mask)
+      (net 1 "GND") (pinfunction "E") (pintype "passive"))
+    (pad "2" thru_hole oval (at 2.54 2.54 90) (size 1.2 1.2) (drill 0.7) (layers *.Cu *.Mask)
+      (net 7 "Net-(R10-Pad2)") (pinfunction "B") (pintype "passive"))
+    (pad "3" thru_hole oval (at 5.08 0 90) (size 1.2 1.2) (drill 0.7) (layers *.Cu *.Mask)
       (net 8 "Net-(R11-Pad1)") (pinfunction "C") (pintype "passive"))
-    (pad "2" thru_hole oval (at 2.54 2.54 270) (size 1.2 1.2) (drill 0.7) (layers *.Cu *.Mask)
-      (net 7 "Net-(R10-Pad2)") (pinfunction "B") (pintype "input"))
-    (pad "3" thru_hole oval (at 5.08 0 270) (size 1.2 1.2) (drill 0.7) (layers *.Cu *.Mask)
-      (net 1 "GND") (pinfunction "E") (pintype "passive"))
-    (model "${KICAD6_3DMODEL_DIR}/Package_TO_SOT_THT.3dshapes/TO-39-3.wrl"
+    (model "${KICAD6_3DMODEL_DIR}/Package_TO_SOT_THT.3dshapes/TO-5-3.wrl"
       (offset (xyz 0 0 0))
       (scale (xyz 1 1 1))
@@
     (effects (font (size 1.5 1.5) (thickness 0.15)))
   )
-  (gr_text "29.11.2022\nboert\nv2" (at 116.84 59.944) (layer "F.SilkS")
+  (gr_text "28.12.2022\nboert\nv3" (at 116.84 59.944) (layer "F.SilkS")
     (effects (font (size 1.5 1.5) (thickness 0.15)))
   )
@@
   (segment (start 179.06 130.815) (end 182.88 130.81) (width 0.4) (layer "B.Cu") (net 6))
   (segment (start 182.88 135.89) (end 190.754 138.43) (width 0.4) (layer "B.Cu") (net 6))
-  (segment (start 191.516 105.41) (end 194.056 107.95) (width 0.4) (layer "B.Cu") (net 7))
-  (segment (start 184.15 105.41) (end 191.516 105.41) (width 0.4) (layer "B.Cu") (net 7))
+  (segment (start 191.606 105.5) (end 194.056 107.95) (width 0.4) (layer "B.Cu") (net 7))
+  (segment (start 189.23 105.5) (end 191.606 105.5) (width 0.4) (layer "B.Cu") (net 7))
   (segment (start 186.69 102.87) (end 193.548 92.71) (width 0.4) (layer "B.Cu") (net 8))
   (segment (start 167.005 127) (end 157.48 127) (width 0.4) (layer "F.Cu") (net 9))
