File: Leiterplatte/Melodieklingel_FA86.kicad_sch (KiCad schematic)
At the start: 47 parts, among them SW1 Taster

Commit message: Leiterplatte v2, mit Korrekturen
Connections:
- net at D100.5: now also TP102.1; no longer R101.1
- net at D100.6: now also R101.1; no longer TP102.1
Other:
- note added: "Anpassung für spannungsführende Klingelleitungen Schaltschwelle: ca. 1,4V"
- note added: "Ergänzung: galvanisch getrennter Eingang Schaltschwelle: ca. 8V (DC) oder 5,6V (AC)"
- note added: "alternativ mit TP3 verbinden und R7 auf 47 kOhm erhöhen"
- note added: "z.B. SC236, SF126, SF136, SF357, SS125 oder SS216"
- note removed: "Anpassung für spannungsführende Klingelleitungen"
- note removed: "Ergänzung: galvanisch getrennter Eingang"
- note removed: "alternativ mit TP3 verbinden"
- moved on the sheet: R101, TP102
Changed lines of the file:
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@@
   (title_block
     (title "Melodieklingel")
-    (date "15.11.22")
-    (rev "1")
+    (date "29.11.22")
+    (rev "2")
     (company "FA 4/86")
     (comment 1 "boert")
@@
     (stroke (width 0) (type default) (color 0 0 0 0))
   )
-  (wire (pts (xy 77.47 195.58) (xy 77.47 196.85))
+  (wire (pts (xy 81.28 193.04) (xy 81.28 196.85))
     (stroke (width 0) (type default) (color 0 0 0 0))
   )
@@
     (stroke (width 0) (type default) (color 0 0 0 0))
   )
-  (wire (pts (xy 77.47 201.93) (xy 77.47 203.2))
+  (wire (pts (xy 81.28 201.93) (xy 81.28 203.2))
     (stroke (width 0) (type default) (color 0 0 0 0))
   )
@@
     (stroke (width 0) (type default) (color 0 0 0 0))
   )
+  (wire (pts (xy 71.12 193.04) (xy 81.28 193.04))
+    (stroke (width 0) (type default) (color 0 0 0 0))
+  )
   (wire (pts (xy 185.42 77.47) (xy 185.42 83.82))
     (stroke (width 0) (type default) (color 0 0 0 0))
@@
     (stroke (width 0) (type default) (color 0 0 0 0))
   )
+  (wire (pts (xy 77.47 190.5) (xy 77.47 195.58))
+    (stroke (width 0) (type default) (color 0 0 0 0))
+  )
   (wire (pts (xy 156.21 39.37) (xy 156.21 69.85))
     (stroke (width 0) (type default) (color 0 0 0 0))
@@
     (stroke (width 0) (type default) (color 0 0 0 0))
   )
-  (wire (pts (xy 71.12 193.04) (xy 74.93 193.04))
+  (wire (pts (xy 71.12 195.58) (xy 77.47 195.58))
     (stroke (width 0) (type default) (color 0 0 0 0))
   )
@@
   )
   (wire (pts (xy 128.27 90.17) (xy 133.35 90.17))
-    (stroke (width 0) (type default) (color 0 0 0 0))
-  )
-  (wire (pts (xy 71.12 195.58) (xy 77.47 195.58))
     (stroke (width 0) (type default) (color 0 0 0 0))
   )
@@
     (effects (font (size 1.27 1.27)) (justify left bottom))
   )
-  (text "Ergänzung:\ngalvanisch getrennter Eingang" (at 25.4 181.61 0)
+  (text "Ergänzung:\ngalvanisch getrennter Eingang\nSchaltschwelle: ca. 8V (DC) oder 5,6V (AC)"
+    (at 25.4 182.88 0)
     (effects (font (size 1.27 1.27)) (justify left bottom))
   )
@@
     (effects (font (size 1.27 1.27)) (justify left bottom))
   )
-  (text "alternativ mit\nTP3 verbinden" (at 72.39 187.96 0)
+  (text "alternativ mit\nTP3 verbinden und\nR7 auf 47 kOhm erhöhen"
+    (at 82.55 187.96 0)
     (effects (font (size 1.27 1.27)) (justify left bottom))
   )
-  (text "Anpassung für spannungsführende\nKlingelleitungen" (at 39.37 166.37 0)
+  (text "Anpassung für spannungsführende\nKlingelleitungen\nSchaltschwelle: ca. 1,4V"
+    (at 35.56 168.91 0)
     (effects (font (size 1.27 1.27)) (justify left bottom))
   )
   (text "Taktgenerator\n" (at 34.29 105.41 0)
+    (effects (font (size 1.27 1.27)) (justify left bottom))
+  )
+  (text "z.B. SC236, SF126,\nSF136, SF357, \nSS125 oder SS216"
+    (at 72.39 161.29 0)
     (effects (font (size 1.27 1.27)) (justify left bottom))
   )
@@
       (effects (font (size 1.27 1.27)) (justify left))
     )
-    (property "Value" "470nF" (id 1) (at 54.3941 80.4485 0)
+    (property "Value" "470pF" (id 1) (at 54.3941 80.4485 0)
       (effects (font (size 1.27 1.27)) (justify left))
     )
@@
     (pin "2")
   )
-  (symbol (lib_id "power:GND") (at 77.47 203.2 0) (unit 1)
-    (in_bom yes) (on_board yes) (fields_autoplaced)
-    (property "Reference" "#PWR0136" (id 0) (at 77.47 209.55 0)
-      (effects (font (size 1.27 1.27)) hide)
-    )
-    (property "Value" "GND" (id 1) (at 77.47 207.6434 0))
-    (property "Footprint" "" (id 2) (at 77.47 203.2 0)
-      (effects (font (size 1.27 1.27)) hide)
-    )
-    (property "Datasheet" "" (id 3) (at 77.47 203.2 0)
+  (symbol (lib_id "power:GND") (at 81.28 203.2 0) (unit 1)
+    (in_bom yes) (on_board yes) (fields_autoplaced)
+    (property "Reference" "#PWR0136" (id 0) (at 81.28 209.55 0)
+      (effects (font (size 1.27 1.27)) hide)
+    )
+    (property "Value" "GND" (id 1) (at 81.28 207.6434 0))
+    (property "Footprint" "" (id 2) (at 81.28 203.2 0)
+      (effects (font (size 1.27 1.27)) hide)
+    )
+    (property "Datasheet" "" (id 3) (at 81.28 203.2 0)
       (effects (font (size 1.27 1.27)) hide)
     )
@@
     (pin "1")
   )
-  (symbol (lib_id "Device:R_Small") (at 77.47 199.39 0) (unit 1)
-    (in_bom yes) (on_board yes) (fields_autoplaced)
-    (property "Reference" "R101" (id 0) (at 78.9686 198.5553 0)
-      (effects (font (size 1.27 1.27)) (justify left))
-    )
-    (property "Value" "1M" (id 1) (at 78.9686 201.0922 0)
-      (effects (font (size 1.27 1.27)) (justify left))
-    )
-    (property "Footprint" "Resistor_THT:R_Axial_DIN0207_L6.3mm_D2.5mm_P5.08mm_Vertical" (id 2) (at 77.47 199.39 0)
-      (effects (font (size 1.27 1.27)) hide)
-    )
-    (property "Datasheet" "~" (id 3) (at 77.47 199.39 0)
+  (symbol (lib_id "Device:R_Small") (at 81.28 199.39 0) (unit 1)
+    (in_bom yes) (on_board yes) (fields_autoplaced)
+    (property "Reference" "R101" (id 0) (at 82.7786 198.5553 0)
+      (effects (font (size 1.27 1.27)) (justify left))
+    )
+    (property "Value" "1M" (id 1) (at 82.7786 201.0922 0)
+      (effects (font (size 1.27 1.27)) (justify left))
+    )
+    (property "Footprint" "Resistor_THT:R_Axial_DIN0207_L6.3mm_D2.5mm_P5.08mm_Vertical" (id 2) (at 81.28 199.39 0)
+      (effects (font (size 1.27 1.27)) hide)
+    )
+    (property "Datasheet" "~" (id 3) (at 81.28 199.39 0)
       (effects (font (size 1.27 1.27)) hide)
     )
@@
     (pin "1")
   )
-  (symbol (lib_id "Connector:TestPoint_Alt") (at 74.93 193.04 270) (unit 1)
+  (symbol (lib_id "Connector:TestPoint_Alt") (at 77.47 190.5 0) (unit 1)
     (in_bom no) (on_board yes)
-    (property "Reference" "TP102" (id 0) (at 76.2 191.262 90)
-      (effects (font (size 1.27 1.27)) (justify left))
-    )
-    (property "Value" "Ausgang" (id 1) (at 76.5298 194.437 0)
+    (property "Reference" "TP102" (id 0) (at 73.66 184.15 0)
+      (effects (font (size 1.27 1.27)) (justify left))
+    )
+    (property "Value" "Ausgang" (id 1) (at 78.867 188.9002 0)
       (effects (font (size 1.27 1.27)) (justify left) hide)
     )
-    (property "Footprint" "TestPoint:TestPoint_THTPad_2.5x2.5mm_Drill1.2mm" (id 2) (at 74.93 198.12 0)
-      (effects (font (size 1.27 1.27)) hide)
-    )
-    (property "Datasheet" "~" (id 3) (at 74.93 198.12 0)
+    (property "Footprint" "TestPoint:TestPoint_THTPad_2.5x2.5mm_Drill1.2mm" (id 2) (at 82.55 190.5 0)
+      (effects (font (size 1.27 1.27)) hide)
+    )
+    (property "Datasheet" "~" (id 3) (at 82.55 190.5 0)
       (effects (font (size 1.27 1.27)) hide)
     )
@@
     )
     (path "/6b3dd195-85f4-4d0b-8872-9b0e0fcca401"
-      (reference "C1") (unit 1) (value "470nF") (footprint "Capacitor_THT:C_Rect_L18.0mm_W7.0mm_P15.00mm_FKS3_FKP3")
+      (reference "C1") (unit 1) (value "470pF") (footprint "Capacitor_THT:C_Rect_L18.0mm_W7.0mm_P15.00mm_FKS3_FKP3")
     )
     (path "/f5f205a8-38dd-49fa-9110-f91b47446353"

Commit message: fix: VT2, Footprint
Parts:
- Q: renamed from VT2; footprint Package_TO_SOT_THT:TO-39-3 -> Package_TO_SOT_THT:TO-5-3
Connections:
- net GND: now also Q.1 (E); no longer Q.3 (E)
- net at R11.1: now also Q.3 (C); no longer Q.1 (C)
Changed lines of the file:
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@@
   (title_block
     (title "Melodieklingel")
-    (date "29.11.22")
-    (rev "2")
+    (date "28.12.22")
+    (rev "3")
     (company "FA 4/86")
     (comment 1 "boert")
@@
     (pin "7")
   )
-  (symbol (lib_id "RFT_Transistoren_und_Dioden:SF126") (at 182.88 99.06 0) (unit 1)
+  (symbol (lib_name "SF126_1") (lib_id "RFT_Transistoren_und_Dioden:SF126") (at 182.88 99.06 0) (unit 1)
     (in_bom yes) (on_board yes) (fields_autoplaced)
     (property "Reference" "VT2" (id 0) (at 187.7314 98.2253 0)
@@
       (effects (font (size 1.27 1.27)) (justify left))
     )
-    (property "Footprint" "Package_TO_SOT_THT:TO-39-3" (id 2) (at 187.96 96.52 0)
-      (effects (font (size 1.27 1.27)) hide)
-    )
-    (property "Datasheet" "" (id 3) (at 182.88 110.49 0)
-      (effects (font (size 1.27 1.27)) hide)
-    )
-    (property "Datasheet" "" (id 4) (at 182.88 99.06 0)
-      (effects (font (size 1.27 1.27)) hide)
-    )
-    (property "Reference" "VT2" (id 5) (at 182.88 99.06 0)
+    (property "Footprint" "Package_TO_SOT_THT:TO-5-3" (id 2) (at 187.96 96.52 0)
+      (effects (font (size 1.27 1.27)) hide)
+    )
+    (property "Datasheet" "https://www.tu-chemnitz.de/etit/zentral/ddr/sf126.gif" (id 3) (at 182.88 110.49 0)
+      (effects (font (size 1.27 1.27)) hide)
+    )
+    (property "Datasheet" "https://www.tu-chemnitz.de/etit/zentral/ddr/sf126.gif" (id 4) (at 182.88 99.06 0)
+      (effects (font (size 1.27 1.27)) hide)
+    )
+    (property "Reference" "Q" (id 5) (at 182.88 99.06 0)
       (effects (font (size 1.27 1.27)) hide)
     )
@@
     )
     (path "/7ee0f32e-5aef-4a7d-9960-e0b6c30786bf"
-      (reference "VT2") (unit 1) (value "SF126") (footprint "Package_TO_SOT_THT:TO-39-3")
-    )
-  )
+      (reference "VT2") (unit 1) (value "SF126") (footprint "Package_TO_SOT_THT:TO-5-3")
+    )
+  )
